File: Hardware/ChibiArmlet.sch (KiCad schematic (older format))
At the start: 38 parts

Commit message: First version of sch ready.
Parts:
- removed C10: 0.1u, CAP_0603, symbol C
- removed C11, C16: 4.7u, CAP_0603, symbol C
- removed C13: 1n, CAP_0603, symbol C
- removed C14: 1u, CAP_0603, symbol C
- removed R2: 100R, RES_0603, symbol R
- removed XL1: CONN_2, symbol CONN_2
- added B1, B2: BAT, symbol BAT
- added BLN1: 0896BM15A0001, symbol BALUN868JOHANSON
- added BZ1: BUZZER, symbol BUZZER
- added C17: 10u, CAP_0805, symbol C
- added C18, C20: 0.1u, symbol C
- added C19, C21: 10u, symbol C
- added D1: BAT54WS, ~, symbol D_SHOTTKY
- added D2: BAT54WS, symbol D_SHOTTKY
- added DA1: NCP1400, symbol NCP1400
- added L1: 5.6nH, IND_0402, symbol L
- added L2: 22uH, symbol L
- added M1: MOTOR, symbol MOTOR
- added Q1, Q2: MMBT2222, symbol NPN
- added Q3: LED_RGB 5050, symbol LED_RGB
- added R10, R8, R9: 51R, RES_0603, symbol R
- added R4: 1k, symbol R
- added R5: 4K7, RES_0402, symbol R
- added R7: 150, RES_0603, symbol R
- added SW1, SW2, SW3: BUTTON, symbol BUTTON
- added XL2: CONN_3, ~, symbol CONN_3
- added XL3: CONN_NOKIA_LCD10, ~, symbol CONN_NOKIA_LCD10
- added XL4: CONN_4, symbol CONN_4
- C1: renamed from C?; value 6.8pF -> 1.8pF
- C11: renamed from C22; value 4.7u -> 10u
- R3: value 100R -> 1k; footprint RES_0603 -> (none)
- R6: value 100R -> 4K7; footprint RES_0603 -> RES_0402
- gave numbers to parts that had none: 16
- renumbered C4 to C12, C6 to C13, C7 to C14, C8 to C15, C9 to C16, DD1 to DD2, XL2 to XL1
Connections:
- net labels added: Btn1, Btn2, Btn3, Buzzer, BuzzerOut, LCD_BCKLT, LCD_SCLK, LCD_SDA, LCD_XCS, LCD_XRES, Lout, P_SCL, P_SDA, PeriphPwr, PeriphPwr1, UART_RX, UART_TX, Vibro, VibroOut
- net labels removed: +5V, DBG_UART_TX
- wire segments 105 -> 193
- no-connect marks 21 -> 11
Other:
- note added: "2xAAA"
- note added: "500R07S1R8BV4"
- note added: "Debug port"
- note added: "L-07C5N6SV4"
- note added: "LCD"
- note added: "Peripheral\nI2C Pull-Ups"
- note added: "Pill"
- note added: "Pill \nConnector"
- note added: "Vibro & buzzer"
- note removed: "Debug port & stuff"
- moved on the sheet: C1, C10, C11, C12, C13, C14, C15, C16, C2, C3, C4, C5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

Commit message: Crystal added
Parts:
- added C22, C23: 15pF, CAP_0402, symbol C
- added R11: 330k*, RES_0402, symbol R
- added R?: 1k, RES_0402, symbol R
- added XTAL2: 32768Hz, KX-26, symbol CRYSTAL_H
- R1: footprint RES_0603 -> RES_0402
Connections:
- wire segments 193 -> 205
- no-connect marks 11 -> 7
Other:
- moved on the sheet: C11, C12, C13, C14, C15, C16, R1

Commit message: Still L MCU
Parts:
- removed ANT1: ANT_PCB_MONO, symbol ANT_PCB_MONO
- added ANT1: ANT_PCB_MONO_2PIN, ~, symbol ANT_PCB_MONO_2PIN
- gave numbers to parts that had none: 1
Connections:
- wire segments 205 -> 206

Commit message: Switch to stm32f051
Parts:
- removed C14: 0.1u, CAP_0603, symbol C
- removed DD2: STM32L151-48, symbol STM32L151-48
- removed R11: 330k*, RES_0402, symbol R
- removed R12: 1k, RES_0402, symbol R
- added B1: BAT, symbol BAT
- added C1: 100pF, CAP_0402, symbol C
- added C20: 0.1u, CAP_0603, symbol C
- added DD1: STM32F051C8, ~, symbol STM32F051C8
- added DD3: M24C02, SO8, symbol EEPROM_I2C
- added F1: FUSE0R, ~, symbol FUSE0R
- C12: renamed from C11; footprint CAP_0603 -> CAP_0805
- C13: renamed from C12; footprint CAP_0603 -> CAP_0402
- C14: renamed from C13; footprint CAP_0603 -> CAP_0402
- C15: value 0.1u -> 10n; footprint CAP_0603 -> CAP_0402
- C16: footprint CAP_0603 -> CAP_0402
- renumbered B1 to B3, C9 to C10, C10 to C11, C22 to C17, C23 to C18, C17 to C19, C1 to C2, C18 to C21, C19 to C22, C20 to C23, C21 to C24, C2 to C3, C3 to C4, C4 to C5, C5 to C6, C6 to C7, C7 to C8, C8 to C9, DD1 to DD2
Connections:
- wire segments 206 -> 213
- no-connect marks 7 -> 11
Other:
- note added: "I2C Addr = 1010 (A2)(A1)(A0) = 1010 111"
- moved on the sheet: ANT1, C12, C13, C14, C15, C16, C17, C18, C2, R1, SW1, SW2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

Commit message: Firefly4 with LQFP-48
Parts:
- removed B1, B2: BAT, symbol BAT
- removed C18: 15pF, CAP_0402, symbol C
- removed C19: 10u, CAP_0805, symbol C
- removed C20: 0.1u, CAP_0603, symbol C
- removed D1: BAT54WS, ~, symbol D_SHOTTKY
- removed DD3: M24C02, SO8, symbol EEPROM_I2C
- removed F1: FUSE0R, ~, symbol FUSE0R
- removed M1: MOTOR, symbol MOTOR
- removed Q1: MMBT2222, symbol NPN
- removed R3: 1k, symbol R
- removed SW1, SW2, SW3: BUTTON, symbol BUTTON
- removed XL3: CONN_NOKIA_LCD10, ~, symbol CONN_NOKIA_LCD10
- removed XTAL2: 32768Hz, KX-26, symbol CRYSTAL_H
- C17: value 15pF -> 10u; footprint CAP_0402 -> CAP_0805
Connections:
- net labels removed: Btn1, Btn2, Btn3, LCD_BCKLT, LCD_SCLK, LCD_SDA, LCD_XCS, LCD_XRES, Vibro, VibroOut
- wire segments 213 -> 152
- no-connect marks 11 -> 22
Other:
- note added: "1xAAA"
- note removed: "2xAAA"
- note removed: "I2C Addr = 1010 (A2)(A1)(A0) = 1010 111"
- note removed: "LCD"
- note removed: "Vibro & buzzer"
- moved on the sheet: BZ1, C12, C13, C14, C15, C16, Q2, R1, R4

Commit message: stm32f050f4 try. No success - pin count is not enough to implement i2c pill.
Parts:
- removed C14: 0.1u, CAP_0402, symbol C
- removed DD1: STM32F051C8, ~, symbol STM32F051C8
- removed TP2: TESTPOINT, symbol TESTPOINT
- added DD?: STM32F05XF4_6, ~, symbol STM32F05XF4_6
Connections:
- net labels removed: CC_GDO2
- wire segments 152 -> 143
- no-connect marks 22 -> 2
Other:
- moved on the sheet: C12, C13, C15, C16, R1, XL1, XL2

Commit message: Software-I2C can be implemented
Parts:
- removed XL2: CONN_3, ~, symbol CONN_3
- added XL?: CONN_2, ~, symbol CONN_2
Connections:
- net labels removed: PeriphPwr, UART_RX
- wire segments 143 -> 140
Changed lines of the file:
@@
 Text Label 6250 1950 0    60   ~ 0
 CC_GDO0
-Text Label 6250 2900 0    60   ~ 0
+Text Label 6250 2500 0    60   ~ 0
 CC_CS
 Text Label 6250 2050 0    60   ~ 0
@@
 	-1   0    0    1
 $EndComp
-Text Label 3200 8050 0    60   ~ 0
-PeriphPwr
-Text Label 1950 1850 0    60   ~ 0
+Text Label 6250 2900 0    60   ~ 0
 P_SCL
-Text Label 1950 1950 0    60   ~ 0
+Text Label 6250 3000 0    60   ~ 0
 P_SDA
-Text Label 1950 1750 0    60   ~ 0
-PeriphPwr
 $Comp
 L BUZZER BZ1
@@
 Text Notes 1750 7850 0    60   Italic 12
 Pill
-Text Label 6350 2500 0    60   ~ 0
-UART_RX
-Text Label 1850 7150 0    60   ~ 0
+Text Label 1850 7050 0    60   ~ 0
 UART_TX
-Text Label 1850 7050 0    60   ~ 0
-UART_RX
-$Comp
-L CONN_3 XL2
-U 1 1 526728AC
-P 1400 7150
-F 0 "XL2" V 1350 7150 40  0000 C CNN
-F 1 "CONN_3" V 1450 7150 40  0000 C CNN
-F 2 "~" H 1400 7150 60  0000 C CNN
-F 3 "~" H 1400 7150 60  0000 C CNN
-	1    1400 7150
-	1    0    0    1
-$EndComp
 Text Notes 6050 9850 0    60   ~ 0
 1xAAA
@@
 	1850 6050 1950 6050
 Wire Wire Line
-	1600 7050 1850 7050
-Wire Wire Line
 	2650 3750 2650 3850
 Wire Wire Line
@@
 	6250 1950 6150 1950
 Wire Wire Line
-	6150 2900 6250 2900
+	6150 2500 6250 2500
 Wire Wire Line
 	6250 2050 6150 2050
@@
 Wire Wire Line
 	3050 8750 3050 8600
-Wire Wire Line
-	2450 1850 1950 1850
-Wire Wire Line
-	2450 1950 1950 1950
-Wire Wire Line
-	1950 1750 2450 1750
 Connection ~ 13650 6300
 Wire Wire Line
@@
 	4150 8600 16000 8600
 Wire Wire Line
-	6350 2500 6150 2500
-Wire Wire Line
-	1850 7150 1600 7150
+	1850 7050 1600 7050
 Wire Wire Line
 	6250 10300 7650 10300
@@
 	6600 1550 6150 1550
 NoConn ~ 10150 2500
+$Comp
+L +3.3V #PWR?
+U 1 1 526D808A
+P 3200 8050
+F 0 "#PWR?" H 3200 8010 30  0001 C CNN
+F 1 "+3.3V" H 3280 8080 30  0000 C CNN
+F 2 "" H 3200 8050 60  0000 C CNN
+F 3 "" H 3200 8050 60  0000 C CNN
+	1    3200 8050
+	1    0    0    -1
+$EndComp
+Wire Wire Line
+	6150 2900 6250 2900
+Wire Wire Line
+	6250 3000 6150 3000
+$Comp
+L CONN_2 XL?
+U 1 1 526D8351
+P 1400 7150
+F 0 "XL?" V 1350 7150 40  0000 C CNN
+F 1 "CONN_2" V 1450 7150 40  0000 C CNN
+F 2 "~" H 1400 7150 60  0000 C CNN
+F 3 "~" H 1400 7150 60  0000 C CNN
+	1    1400 7150
+	-1   0    0    -1
+$EndComp
 $EndSCHEMATC
