File: Hardware/ChibiArmlet.sch (KiCad schematic (older format))
At the start: 52 parts, among them Q2 MMBT2222, Q3 LED_RGB 5050

Commit message: MCU replaced with stm32L100c6
Parts:
- removed DD1: STM32F051C8, ~, symbol STM32F051C8
- added C?: 0.1u, CAP_0402, symbol C
- added DD?: STM32L100CX, ~, symbol STM32L100CX
Connections:
- wire segments 152 -> 156
- no-connect marks 22 -> 21
Other:
- moved on the sheet: C12, C13, C14, C15, C16, R1

Commit message: Again, buttons and display added.
Parts:
- added R3: 51R, RES_0603, symbol R
- added SW1, SW2, SW3: BUTTON, ~, symbol BUTTON
- added XL3: CONN_NOKIA_LCD10, symbol CONN_NOKIA_LCD10
- gave numbers to parts that had none: 2
Connections:
- net labels added: BTN1, BTN2, BTN3, LCD_BCKLT, LCD_SCLK, LCD_SDA, LCD_XCS, LCD_XRES
- wire segments 156 -> 183
- no-connect marks 21 -> 13
Other:
- note added: "LCD"
Changed lines of the file:
@@
 Sheet 1 1
 Title ""
-Date "28 oct 2013"
+Date "29 oct 2013"
 Rev ""
 Comp ""
@@
 Comment4 ""
 $EndDescr
-NoConn ~ 3800 1600
 Text Notes 1350 6700 0    60   Italic 12
 Debug port
@@
 Text Notes 12200 10950 0    60   Italic 12
 WWPASS Reader G.II
-NoConn ~ 3800 1500
 Text Label 3650 1300 2    60   ~ 0
 BLUE_LED
@@
 	1    0    0    -1
 $EndComp
-Text Label 3350 2300 0    60   ~ 0
+Text Label 3350 1600 0    60   ~ 0
 Buzzer
 Text Notes 1750 7850 0    60   Italic 12
@@
 	13650 6850 13650 6950
 Wire Wire Line
-	3350 2300 3800 2300
+	3350 1600 3800 1600
 Wire Notes Line
 	450  4900 16050 4900
@@
 Wire Wire Line
 	6250 10300 6250 10350
-NoConn ~ 6450 1400
 NoConn ~ 6450 2100
 NoConn ~ 6450 2400
@@
 NoConn ~ 6450 3650
 NoConn ~ 3800 1700
-NoConn ~ 3800 2400
-NoConn ~ 3800 2500
-NoConn ~ 3800 2600
-NoConn ~ 3800 2700
-NoConn ~ 3800 2800
-$Comp
-L STM32L100CX DD?
+$Comp
+L STM32L100CX DD1
 U 1 1 526E377D
 P 5100 2500
-F 0 "DD?" H 4600 3850 60  0000 C CNN
+F 0 "DD1" H 4600 3850 60  0000 C CNN
 F 1 "STM32L100CX" H 5250 3850 60  0000 C CNN
 F 2 "~" H 5100 2500 60  0000 C CNN
@@
 	3150 3700 3150 3350
 $Comp
-L GND #PWR?
+L GND #PWR049
 U 1 1 526E3E25
 P 2900 4200
-F 0 "#PWR?" H 2990 4180 30  0001 C CNN
+F 0 "#PWR049" H 2990 4180 30  0001 C CNN
 F 1 "GND" H 2900 4120 30  0001 C CNN
 F 2 "" H 2900 4200 60  0001 C CNN
@@
 $EndComp
 $Comp
-L C C?
+L C C18
 U 1 1 526E3E2B
 P 2900 3900
-F 0 "C?" H 2800 3800 50  0000 L CNN
+F 0 "C18" H 2800 3800 50  0000 L CNN
 F 1 "0.1u" H 2800 4000 50  0000 L CNN
 F 2 "CAP_0402" V 3000 3750 28  0000 C BNN
@@
 	2900 4100 2900 4200
 $Comp
-L +3.3V #PWR?
+L +3.3V #PWR050
 U 1 1 526E3E32
 P 2850 3250
-F 0 "#PWR?" H 2850 3210 30  0001 C CNN
+F 0 "#PWR050" H 2850 3210 30  0001 C CNN
 F 1 "+3.3V" H 2930 3280 30  0000 C CNN
 F 2 "" H 2850 3250 60  0001 C CNN
@@
 	2650 3700 2650 3150
 Connection ~ 2650 3150
+$Comp
+L GND #PWR051
+U 1 1 5270301A
+P 6250 7100
+F 0 "#PWR051" H 6340 7080 30  0001 C CNN
+F 1 "GND" H 6250 7020 30  0001 C CNN
+F 2 "" H 6250 7100 60  0000 C CNN
+F 3 "" H 6250 7100 60  0000 C CNN
+	1    6250 7100
+	1    0    0    -1
+$EndComp
+$Comp
+L BUTTON SW1
+U 1 1 52703029
+P 5850 6200
+F 0 "SW1" H 5650 6350 50  0000 C CNN
+F 1 "BUTTON" H 5950 6350 50  0000 C CNN
+F 2 "~" H 5850 6200 60  0000 C CNN
+F 3 "~" H 5850 6200 60  0000 C CNN
+	1    5850 6200
+	1    0    0    -1
+$EndComp
+$Comp
+L BUTTON SW2
+U 1 1 52703038
+P 5850 6550
+F 0 "SW2" H 5650 6700 50  0000 C CNN
+F 1 "BUTTON" H 5950 6700 50  0000 C CNN
+F 2 "~" H 5850 6550 60  0000 C CNN
+F 3 "~" H 5850 6550 60  0000 C CNN
+	1    5850 6550
+	1    0    0    -1
+$EndComp
+$Comp
+L BUTTON SW3
+U 1 1 52703047
+P 5850 6900
+F 0 "SW3" H 5650 7050 50  0000 C CNN
+F 1 "BUTTON" H 5950 7050 50  0000 C CNN
+F 2 "~" H 5850 6900 60  0000 C CNN
+F 3 "~" H 5850 6900 60  0000 C CNN
+	1    5850 6900
+	1    0    0    -1
+$EndComp
+Wire Wire Line
+	6250 7100 6250 6200
+Wire Wire Line
+	6250 6200 6150 6200
+Wire Wire Line
+	6150 6550 6250 6550
+Connection ~ 6250 6550
+Wire Wire Line
+	6150 6900 6250 6900
+Connection ~ 6250 6900
+Text Label 5200 6200 0    60   ~ 0
+BTN1
+Text Label 5200 6550 0    60   ~ 0
+BTN2
+Text Label 5200 6900 0    60   ~ 0
+BTN3
+Wire Wire Line
+	5550 6200 5200 6200
+Wire Wire Line
+	5550 6550 5200 6550
+Wire Wire Line
+	5550 6900 5200 6900
+Text Label 6500 1400 0    60   ~ 0
+BTN1
+Text Label 3550 1500 0    60   ~ 0
+BTN2
+Text Label 3550 2800 0    60   ~ 0
+BTN3
+$Comp
+L GND #PWR052
+U 1 1 52704227
+P 8350 7100
+F 0 "#PWR052" H 8440 7080 30  0001 C CNN
+F 1 "GND" H 8350 7020 30  0001 C CNN
+F 2 "" H 8350 7100 60  0001 C CNN
+F 3 "" H 8350 7100 60  0001 C CNN
+	1    8350 7100
+	0    -1   -1   0
+$EndComp
+Text Notes 7400 6700 0    60   ~ 0
+LCD
+$Comp
+L +3.3V #PWR053
+U 1 1 5270422E
+P 8500 6700
+F 0 "#PWR053" H 8500 6660 30  0001 C CNN
+F 1 "+3.3V" H 8580 6730 30  0000 C CNN
+F 2 "" H 8500 6700 60  0001 C CNN
+F 3 "" H 8500 6700 60  0001 C CNN
+	1    8500 6700
+	1    0    0    -1
+$EndComp
+$Comp
+L GND #PWR054
+U 1 1 52704234
+P 8350 6850
+F 0 "#PWR054" H 8440 6830 30  0001 C CNN
+F 1 "GND" H 8350 6770 30  0001 C CNN
+F 2 "" H 8350 6850 60  0001 C CNN
+F 3 "" H 8350 6850 60  0001 C CNN
+	1    8350 6850
+	0    -1   -1   0
+$EndComp
+Text Label 9150 7000 0    60   ~ 0
+LCD_BCKLT
+Text Label 8400 6150 0    60   ~ 0
+LCD_SCLK
+Text Label 8400 6250 0    60   ~ 0
+LCD_SDA
+Text Label 8400 6350 0    60   ~ 0
+LCD_XCS
+Text Label 8400 6450 0    60   ~ 0
+LCD_XRES
+Text Label 3350 2500 0    60   ~ 0
+LCD_SCLK
+Text Label 3350 2300 0    60   ~ 0
+LCD_SDA
+Text Label 3350 2400 0    60   ~ 0
+LCD_XRES
+Text Label 3350 2600 0    60   ~ 0
+LCD_XCS
+Text Label 3350 2700 0    60   ~ 0
+LCD_BCKLT
+Wire Wire Line
+	3800 2700 3350 2700
+Wire Wire Line
+	3800 2600 3350 2600
+Wire Wire Line
+	3800 2400 3350 2400
+Wire Wire Line
+	3800 2300 3350 2300
+Wire Wire Line
+	3800 2500 3350 2500
+Wire Wire Line
+	8400 6450 8300 6450
+Wire Wire Line
+	8400 6250 8300 6250
+Wire Wire Line
+	8350 7100 8300 7100
+Wire Wire Line
+	8350 6850 8300 6850
+Wire Wire Line
+	8350 6650 8300 6650
+Wire Wire Line
+	8350 6650 8350 6750
+Wire Wire Line
+	8350 6750 8300 6750
+Wire Wire Line
+	8350 6700 8500 6700
+Connection ~ 8350 6700
+Wire Wire Line
+	8300 7000 8500 7000
+Wire Wire Line
+	8300 6150 8400 6150
+Wire Wire Line
+	8300 6350 8400 6350
+$Comp
+L R R3
+U 1 1 52704260
+P 8750 7000
+F 0 "R3" V 8830 6850 50  0000 C CNN
+F 1 "51R" V 8750 7000 50  0000 C CNN
+F 2 "RES_0603" V 8830 7100 28  0000 C CNN
+F 3 "" H 8750 7000 60  0000 C CNN
+	1    8750 7000
+	0    -1   -1   0
+$EndComp
+Wire Wire Line
+	9000 7000 9150 7000
+$Comp
+L CONN_NOKIA_LCD10 XL3
+U 1 1 52704267
+P 8000 6500
+F 0 "XL3" V 7700 6700 60  0000 C CNN
+F 1 "CONN_NOKIA_LCD10" V 7700 6150 60  0000 C CNN
+F 2 "" H 8000 6500 60  0000 C CNN
+F 3 "" H 8000 6500 60  0000 C CNN
+	1    8000 6500
+	1    0    0    -1
+$EndComp
+Wire Wire Line
+	6500 1400 6450 1400
+Wire Wire Line
+	3800 1500 3550 1500
+Wire Wire Line
+	3550 2800 3800 2800
 $EndSCHEMATC

Commit message: PCB routed save antenna. Quartz added.
Parts:
- added C19, C20: 6.8pF, symbol C
- added R11: 200k*, RES_0402, symbol R
- added XTAL2: 32768, symbol CRYSTAL_H
Connections:
- wire segments 183 -> 192
- no-connect marks 13 -> 11

Commit message: + Antenna + Quartz 32768
Parts:
- removed ANT1: ANT_PCB_MONO_2PIN, ~, symbol ANT_PCB_MONO_2PIN
- added ANT1: ANT_PCB_MONO, ~, symbol ANT_PCB_MONO
Connections:
- wire segments 192 -> 191
Changed lines of the file:
@@
 Text Notes 6050 9850 0    60   ~ 0
 1xAAA
-$Comp
-L ANT_PCB_MONO_2PIN ANT1
-U 1 1 526B6399
-P 15200 1950
-F 0 "ANT1" H 15000 2200 60  0000 C CNN
-F 1 "ANT_PCB_MONO_2PIN" H 15350 1650 60  0000 C CNN
-F 2 "~" H 15200 1950 60  0000 C CNN
-F 3 "~" H 15200 1950 60  0000 C CNN
-	1    15200 1950
-	1    0    0    -1
-$EndComp
-$Comp
-L GND #PWR046
-U 1 1 526B63A6
-P 15000 2100
-F 0 "#PWR046" H 15090 2080 30  0001 C CNN
-F 1 "GND" H 15000 2020 30  0001 C CNN
-F 2 "" H 15000 2100 60  0001 C CNN
-F 3 "" H 15000 2100 60  0001 C CNN
-	1    15000 2100
-	1    0    0    -1
-$EndComp
 NoConn ~ 6450 3150
 NoConn ~ 6450 3250
@@
 $EndComp
 $Comp
-L +3.3V #PWR047
+L +3.3V #PWR046
 U 1 1 526D45BA
 P 14800 6300
-F 0 "#PWR047" H 14800 6260 30  0001 C CNN
+F 0 "#PWR046" H 14800 6260 30  0001 C CNN
 F 1 "+3.3V" H 14880 6330 30  0000 C CNN
 F 2 "" H 14800 6300 60  0000 C CNN
@@
 $EndComp
 $Comp
-L GND #PWR048
+L GND #PWR047
 U 1 1 526D45C7
 P 14650 6950
-F 0 "#PWR048" H 14740 6930 30  0001 C CNN
+F 0 "#PWR047" H 14740 6930 30  0001 C CNN
 F 1 "GND" H 14650 6870 30  0001 C CNN
 F 2 "" H 14650 6950 60  0001 C CNN
@@
 NoConn ~ 3800 3500
 $Comp
-L GND #PWR049
+L GND #PWR048
 U 1 1 526E3E25
 P 2900 4200
-F 0 "#PWR049" H 2990 4180 30  0001 C CNN
+F 0 "#PWR048" H 2990 4180 30  0001 C CNN
 F 1 "GND" H 2900 4120 30  0001 C CNN
 F 2 "" H 2900 4200 60  0001 C CNN
@@
 $EndComp
 $Comp
-L +3.3V #PWR050
+L +3.3V #PWR049
 U 1 1 526E3E32
 P 2850 3250
-F 0 "#PWR050" H 2850 3210 30  0001 C CNN
+F 0 "#PWR049" H 2850 3210 30  0001 C CNN
 F 1 "+3.3V" H 2930 3280 30  0000 C CNN
 F 2 "" H 2850 3250 60  0001 C CNN
@@
 $EndComp
 $Comp
-L GND #PWR051
+L GND #PWR050
 U 1 1 5270301A
 P 6250 7100
-F 0 "#PWR051" H 6340 7080 30  0001 C CNN
+F 0 "#PWR050" H 6340 7080 30  0001 C CNN
 F 1 "GND" H 6250 7020 30  0001 C CNN
 F 2 "" H 6250 7100 60  0000 C CNN
@@
 BTN3
 $Comp
-L GND #PWR052
+L GND #PWR051
 U 1 1 52704227
 P 8350 7100
-F 0 "#PWR052" H 8440 7080 30  0001 C CNN
+F 0 "#PWR051" H 8440 7080 30  0001 C CNN
 F 1 "GND" H 8350 7020 30  0001 C CNN
 F 2 "" H 8350 7100 60  0001 C CNN
@@
 LCD
 $Comp
-L +3.3V #PWR053
+L +3.3V #PWR052
 U 1 1 5270422E
 P 8500 6700
-F 0 "#PWR053" H 8500 6660 30  0001 C CNN
+F 0 "#PWR052" H 8500 6660 30  0001 C CNN
 F 1 "+3.3V" H 8580 6730 30  0000 C CNN
 F 2 "" H 8500 6700 60  0001 C CNN
@@
 $EndComp
 $Comp
-L GND #PWR054
+L GND #PWR053
 U 1 1 52704234
 P 8350 6850
-F 0 "#PWR054" H 8440 6830 30  0001 C CNN
+F 0 "#PWR053" H 8440 6830 30  0001 C CNN
 F 1 "GND" H 8350 6770 30  0001 C CNN
 F 2 "" H 8350 6850 60  0001 C CNN
@@
 Wire Wire Line
 	6250 10300 7650 10300
-Wire Wire Line
-	15000 2000 15000 2100
 Connection ~ 3450 3650
 Connection ~ 3700 3650
@@
 $EndComp
 $Comp
-L GND #PWR055
+L GND #PWR054
 U 1 1 5270DB84
 P 7050 4500
-F 0 "#PWR055" H 7140 4480 30  0001 C CNN
+F 0 "#PWR054" H 7140 4480 30  0001 C CNN
 F 1 "GND" H 7050 4420 30  0001 C CNN
 F 2 "" H 7050 4500 60  0001 C CNN
@@
 $EndComp
 $Comp
-L GND #PWR056
+L GND #PWR055
 U 1 1 5270DB8A
 P 7650 4500
-F 0 "#PWR056" H 7740 4480 30  0001 C CNN
+F 0 "#PWR055" H 7740 4480 30  0001 C CNN
 F 1 "GND" H 7650 4420 30  0001 C CNN
 F 2 "" H 7650 4500 60  0001 C CNN
@@
 $EndComp
 $Comp
-L GND #PWR057
+L GND #PWR056
 U 1 1 5270DB90
 P 7350 4500
-F 0 "#PWR057" H 7440 4480 30  0001 C CNN
+F 0 "#PWR056" H 7440 4480 30  0001 C CNN
 F 1 "GND" H 7350 4420 30  0001 C CNN
 F 2 "" H 7350 4500 60  0001 C CNN
@@
 Wire Wire Line
 	6450 3650 6550 3650
+$Comp
+L ANT_PCB_MONO ANT1
+U 1 1 527152AC
+P 15200 1900
+F 0 "ANT1" H 15000 2150 60  0000 C CNN
+F 1 "ANT_PCB_MONO" H 15250 2050 60  0000 C CNN
+F 2 "~" H 15200 1900 60  0000 C CNN
+F 3 "~" H 15200 1900 60  0000 C CNN
+	1    15200 1900
+	1    0    0    -1
+$EndComp
 $EndSCHEMATC

Commit message: Prototype sent to factory
Parts:
- removed C1: 100pF, CAP_0402, symbol C
Connections:
- wire segments 191 -> 190
Other:
- moved on the sheet: ANT1
Changed lines of the file:
@@
 Sheet 1 1
 Title ""
-Date "30 oct 2013"
+Date "31 oct 2013"
 Rev ""
 Comp ""
@@
 NoConn ~ 6450 3450
 $Comp
-L C C1
-U 1 1 526CD506
-P 14700 1900
-F 0 "C1" V 14900 1750 50  0000 L CNN
-F 1 "100pF" V 14900 1900 50  0000 L CNN
-F 2 "CAP_0402" V 14800 1750 28  0000 C BNN
-F 3 "~" H 14700 1900 60  0000 C CNN
-	1    14700 1900
-	0    -1   -1   0
-$EndComp
-$Comp
 L +3.3V #PWR046
 U 1 1 526D45BA
@@
 Connection ~ 3150 3350
 Wire Wire Line
-	15000 1900 14900 1900
-Wire Wire Line
-	14400 1900 14500 1900
+	14400 1900 14600 1900
 Connection ~ 14450 1900
 Wire Wire Line
@@
 L ANT_PCB_MONO ANT1
 U 1 1 527152AC
-P 15200 1900
-F 0 "ANT1" H 15000 2150 60  0000 C CNN
-F 1 "ANT_PCB_MONO" H 15250 2050 60  0000 C CNN
-F 2 "~" H 15200 1900 60  0000 C CNN
-F 3 "~" H 15200 1900 60  0000 C CNN
-	1    15200 1900
-	1    0    0    -1
-$EndComp
+P 14800 1900
+F 0 "ANT1" H 14600 2150 60  0000 C CNN
+F 1 "ANT_PCB_MONO" H 14850 2050 60  0000 C CNN
+F 2 "~" H 14800 1900 60  0000 C CNN
+F 3 "~" H 14800 1900 60  0000 C CNN
+	1    14800 1900
+	1    0    0    -1
+$EndComp

Commit message: + Vibro +Debug Pin * All R 0402 * 10u 0603
Parts:
- removed DD1: STM32L100CX, ~, symbol STM32L100CX
- removed RP3, RP4: REFPOINT, symbol REFPOINT
- removed XTAL2: 32768, symbol CRYSTAL_H
- added C1: 10u, CAP_0603, symbol C
- added D1: BAT54WS, symbol D_SHOTTKY
- added DD1: STM32L151CXTX, ~, symbol STM32L151CXTX
- added M1: MOTOR_PAD, ~, symbol MOTOR_PAD
- added Q1: MMBT2222, symbol NPN
- added R12: 1k, symbol R
- added XL5: CONN_1, ~, symbol CONN_1
- added XTAL2: 32768, KXT26, symbol CRYSTAL
- C12, C17: footprint CAP_0805 -> CAP_0603
- R7: footprint RES_0603 -> RES_0402
Connections:
- net labels added: Vibro, VibroOut
- wire segments 190 -> 203
- no-connect marks 11 -> 8
Other:
- note added: "Debug \nPin"
- moved on the sheet: BZ1, C17, C19, C20, Q2, R11, R4

Commit message: - Buttons - LCD - Quartz 32768
Parts:
- removed C19, C20: 6.8pF, symbol C
- removed R11: 200k*, RES_0402, symbol R
- removed R3: 51R, RES_0603, symbol R
- removed SW1, SW2, SW3: BUTTON, ~, symbol BUTTON
- removed XL3: CONN_NOKIA_LCD10, symbol CONN_NOKIA_LCD10
- removed XTAL2: 32768, KXT26, symbol CRYSTAL
Connections:
- net labels removed: BTN1, BTN2, BTN3, LCD_BCKLT, LCD_SCLK, LCD_SDA, LCD_XCS, LCD_XRES
- wire segments 203 -> 168
- no-connect marks 8 -> 18
Other:
- note removed: "LCD"

Commit message: + 4-pin connector for functionality raising
Parts:
- removed XL5: CONN_1, ~, symbol CONN_1
- added XL3: CONN_4, ~, symbol CONN_4
Connections:
- wire segments 168 -> 171
- no-connect marks 18 -> 16
Other:
- note added: "Just\nPins"
- note removed: "Debug \nPin"
Changed lines of the file:
@@
 Sheet 1 1
 Title ""
-Date "6 dec 2013"
+Date "8 dec 2013"
 Rev ""
 Comp ""
@@
 Wire Wire Line
 	3800 3500 3700 3500
-NoConn ~ 6450 3200
 NoConn ~ 6450 3050
 NoConn ~ 6450 2950
-$Comp
-L CONN_1 XL5
-U 1 1 52A1ABA5
-P 7300 2800
-F 0 "XL5" V 7250 2810 40  0000 C CNN
-F 1 "CONN_1" V 7310 2820 40  0000 C CNN
-F 2 "~" H 7300 2800 60  0000 C CNN
-F 3 "~" H 7300 2800 60  0000 C CNN
-	1    7300 2800
-	1    0    0    -1
-$EndComp
-Wire Wire Line
-	7100 2800 6450 2800
-Text Notes 7400 2800 0    60   ~ 0
-Debug \nPin
+Text Notes 6950 3350 0    60   ~ 0
+Just\nPins
 Connection ~ 15050 5850
 Wire Wire Line
@@
 	15050 5400 15050 5900
 $Comp
-L +BATT #PWR050
-U 1 1 52A1C42B
-P 15100 5850
-F 0 "#PWR050" H 15100 5810 30  0001 C CNN
-F 1 "+BATT" H 15180 5880 30  0000 C CNN
-F 2 "" H 15100 5850 60  0001 C CNN
-F 3 "" H 15100 5850 60  0001 C CNN
-	1    15100 5850
-	1    0    0    -1
-$EndComp
-$Comp
-L GND #PWR051
+L GND #PWR050
 U 1 1 52A1C431
 P 15050 6400
-F 0 "#PWR051" H 15140 6380 30  0001 C CNN
+F 0 "#PWR050" H 15140 6380 30  0001 C CNN
 F 1 "GND" H 15050 6320 30  0001 C CNN
 F 2 "" H 15050 6400 60  0001 C CNN
@@
 $EndComp
 $Comp
-L GND #PWR052
+L GND #PWR051
 U 1 1 52A1C449
 P 13700 6500
-F 0 "#PWR052" H 13790 6480 30  0001 C CNN
+F 0 "#PWR051" H 13790 6480 30  0001 C CNN
 F 1 "GND" H 13700 6420 30  0001 C CNN
 F 2 "" H 13700 6500 60  0001 C CNN
@@
 $EndComp
 $Comp
-L GND #PWR053
+L GND #PWR052
 U 1 1 52A1CB8F
 P 14550 6400
-F 0 "#PWR053" H 14640 6380 30  0001 C CNN
+F 0 "#PWR052" H 14640 6380 30  0001 C CNN
 F 1 "GND" H 14550 6320 30  0001 C CNN
 F 2 "" H 14550 6400 60  0000 C CNN
@@
 Wire Wire Line
 	14550 6400 14550 6250
-NoConn ~ 6450 3400
-NoConn ~ 6450 3300
 NoConn ~ 6450 1400
 NoConn ~ 3800 1500
@@
 NoConn ~ 3800 2700
 NoConn ~ 3800 2800
+$Comp
+L +3.3V #PWR053
+U 1 1 52A1E0A0
+P 15100 5850
+F 0 "#PWR053" H 15100 5810 30  0001 C CNN
+F 1 "+3.3V" H 15180 5880 30  0000 C CNN
+F 2 "" H 15100 5850 60  0000 C CNN
+F 3 "" H 15100 5850 60  0000 C CNN
+	1    15100 5850
+	1    0    0    -1
+$EndComp
+$Comp
+L CONN_4 XL3
+U 1 1 52A4B5B3
+P 6800 3250
+F 0 "XL3" V 6750 3250 40  0000 C CNN
+F 1 "CONN_4" V 6850 3250 40  0000 C CNN
+F 2 "~" H 6800 3250 60  0000 C CNN
+F 3 "~" H 6800 3250 60  0000 C CNN
+	1    6800 3250
+	-1   0    0    1
+$EndComp
+NoConn ~ 6450 2800
+Wire Wire Line
+	6600 3200 6450 3200
+Wire Wire Line
+	6450 3300 6600 3300
+Wire Wire Line
+	6600 3400 6450 3400
+$Comp
+L GND #PWR054
+U 1 1 52A4B8F6
+P 6600 3000
+F 0 "#PWR054" H 6690 2980 30  0001 C CNN
+F 1 "GND" H 6600 2920 30  0001 C CNN
+F 2 "" H 6600 3000 60  0000 C CNN
+F 3 "" H 6600 3000 60  0000 C CNN
+	1    6600 3000
+	1    0    0    -1
+$EndComp
+Wire Wire Line
+	6600 3100 6600 3000
 $EndSCHEMATC
