File: Hardware/ChibiArmlet.sch (KiCad schematic (older format))
At the start: 56 parts, among them M1 MOTOR_PAD, Q1 MMBT2222, Q2 MMBT2222, Q3 LED_RGB 5050

Commit message: Hardware v3, sent to pilot production
Other:
- note added: "1xAA"
- note removed: "1xAAA"
- note removed: "WWPASS Reader G.II"
Changed lines of the file:
@@
 Sheet 1 1
 Title ""
-Date "8 dec 2013"
+Date "10 dec 2013"
 Rev ""
 Comp ""
@@
 Text Notes 5050 700  0    60   Italic 12
 CPU
-Text Notes 1800 9900 0    60   Italic 12
+Text Notes 1800 9900 0    60   ~ 12
 Indication
-Text Notes 7700 9800 0    60   Italic 12
+Text Notes 7700 9800 0    60   ~ 12
 Power
-Text Notes 12200 10950 0    60   Italic 12
-WWPASS Reader G.II
 Text Label 3650 1300 2    60   ~ 0
 BLUE_LED
@@
 $EndComp
 Text Notes 6050 9850 0    60   ~ 0
-1xAAA
+1xAA
 $Comp
 L +3.3V #PWR046
@@
 F 3 "~" H 14550 5850 60  0000 C CNN
 	1    14550 5850
-	-1   0    0    -1
-$EndComp
-$Comp
+	1    0    0    -1
+$EndComp
+$Comp

Commit message: * Vibro disconnected from 3V3, connected to Vbat. * BOM renewed
Changed lines of the file:
@@
 Sheet 1 1
 Title ""
-Date "10 dec 2013"
+Date "29 dec 2013"
 Rev ""
 Comp ""
@@
 NoConn ~ 3800 2800
 $Comp
-L +3.3V #PWR053
-U 1 1 52A1E0A0
-P 15100 5850
-F 0 "#PWR053" H 15100 5810 30  0001 C CNN
-F 1 "+3.3V" H 15180 5880 30  0000 C CNN
-F 2 "" H 15100 5850 60  0000 C CNN
-F 3 "" H 15100 5850 60  0000 C CNN
-	1    15100 5850
-	1    0    0    -1
-$EndComp
-$Comp
 L CONN_4 XL3
 U 1 1 52A4B5B3
@@
 Wire Wire Line
 	6600 3100 6600 3000
+$Comp
+L +BATT #PWR?
+U 1 1 52BFD5E2
+P 15100 5850
+F 0 "#PWR?" H 15100 5810 30  0001 C CNN
+F 1 "+BATT" H 15180 5880 30  0000 C CNN
+F 2 "" H 15100 5850 60  0001 C CNN
+F 3 "" H 15100 5850 60  0001 C CNN
+	1    15100 5850
+	1    0    0    -1
+$EndComp
 $EndSCHEMATC

Commit message: CPU name changed
Parts:
- DD1: symbol STM32L151CXTX -> STM32L151CxTx
Changed lines of the file:
@@
 LIBS:memory
 LIBS:ChibiArmlet-cache
-EELAYER 27 0
+EELAYER 25 0
 EELAYER END
 $Descr A3 16535 11693
@@
 $EndComp
 $Comp
-L STM32L151CXTX DD1
+L STM32L151CxTx DD1
 U 1 1 52A19E0D
 P 5100 2500

Commit message: Some sch changes
Parts:
- ANT1: symbol ANT_PCB_MONO -> Antennas_kl:ANT_PCB_MONO
- B3: symbol BAT -> Power_kl:BAT
- BLN1: symbol BALUN868JOHANSON -> RFICs:BALUN868JOHANSON
- BZ1: symbol BUZZER -> Tittar_kl:BUZZER
- C1, C10, C11, C12, C13, C14, C15, C16, C17, C18, C2, C21, C22, C23, C24, C3, C4, C5, C6, C7, C8, C9: symbol C -> Tittar_kl:C
- D1, D2: symbol D_SHOTTKY -> Tittar_kl:D_Shottky
- DA1: symbol NCP1400 -> Power_kl:NCP1400
- DD1: symbol STM32L151CxTx -> st_kl:STM32L151CxTx
- DD2: symbol CC1101 -> RFICs:CC1101
- L1, L2: symbol L -> Tittar_kl:L
- M1: symbol MOTOR_PAD -> Tittar_kl:MOTOR_PAD
- Q1, Q2: symbol NPN -> Transistors_kl:NPN
- Q3: symbol LED_RGB -> ChibiArmlet-rescue:LED_RGB-RESCUE-ChibiArmlet
- R1, R10, R12, R2, R4, R5, R6, R7, R8, R9: symbol R -> Tittar_kl:R
- RP1, RP2: symbol REFPOINT -> pcb_details:REFPOINT
- TP1, TP2: symbol TESTPOINT -> ChibiArmlet-rescue:TESTPOINT-RESCUE-ChibiArmlet
- XL1: symbol ST_SWD -> Connectors_kl:ST_SWD
- XL2: symbol CONN_3 -> Connectors_kl:CONN_3
- XL3, XL4: symbol CONN_4 -> Connectors_kl:CONN_4
- XTAL1: symbol CRYSTAL_H -> Tittar_kl:CRYSTAL_H
Connections:
- wire segments 171 -> 214
