File: Pill/Pill4.kicad_pcb (KiCad board)
At the start: 2 copper layers, 24.6 x 10.4 mm, 6 parts

Commit message: + Pill4 * Indication added
Routing:
- added copper zone on B.Cu, net GND
- added copper zone on F.Cu, net GND
Changed lines of the file:
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@@
     (links 13)
     (no_connects 0)
-    (area 120.209499 93.409499 145.190501 104.190501)
+    (area 113.685999 92.804144 145.190501 104.190501)
     (thickness 1.6002)
     (drawings 5)
@@
     (last_trace_width 0.2)
     (trace_clearance 0.2)
-    (zone_clearance 0.29972)
+    (zone_clearance 0.3)
     (zone_45_only no)
     (trace_min 0.18034)
@@
     (visible_elements 7FFFFFFF)
     (pcbplotparams
-      (layerselection 276856832)
+      (layerselection 281051137)
       (usegerberextensions true)
       (excludeedgelayer true)
@@
   (segment (start 126.5094 98.8874) (end 127.006 98.8874) (width 0.5) (layer Front) (net 7))
   (segment (start 124.4 97.53) (end 126.5094 98.8874) (width 0.5) (layer Front) (net 7))
+  (zone (net 7) (net_name GND) (layer Front) (hatch edge 0.508)
+    (connect_pads (clearance 0.3))
+    (min_thickness 0.254)
+    (fill (arc_segments 16) (thermal_gap 0.3) (thermal_bridge_width 0.508))
+    (polygon
+      (pts
+        (xy 120.4 93.6) (xy 145 93.6) (xy 145 104) (xy 120.4 104)
+      )
+    )
+  )
+  (zone (net 7) (net_name GND) (layer Back) (hatch edge 0.508)
+    (connect_pads (clearance 0.3))
+    (min_thickness 0.254)
+    (fill (arc_segments 16) (thermal_gap 0.3) (thermal_bridge_width 0.508))
+    (polygon
+      (pts
+        (xy 120.4 93.6) (xy 145 93.6) (xy 145 104) (xy 120.4 104)
+      )
+    )
+  )
 )
